Commit message: sensors added

File: robot/src/robot/urdf/robot.urdf (robot description, URDF)
Before this commit: robot robot, 29 links, 28 joints
Links:
- added link ir_back_center_offset_link
- added link ir_front_center_offset_link
- added link ir_front_left_offset_link
- added link ir_front_right_offset_link
Joints:
- added joint ir_back_center_offset_joint: type fixed, parent ir_back_center_link, child ir_back_center_offset_link, origin xyz=-0.0163 -0.0035 -0.006 rpy=0 0 3.14159
- added joint ir_front_center_offset_joint: type fixed, parent ir_front_center_link, child ir_front_center_offset_link, origin xyz=0.0163 0.0035 -0.006 rpy=0 0 0
- added joint ir_front_left_offset_joint: type fixed, parent ir_front_left_link, child ir_front_left_offset_link, origin xyz=0.012 0.012 -0.006 rpy=0 0 0.55
- added joint ir_front_right_offset_joint: type fixed, parent ir_front_right_link, child ir_front_right_offset_link, origin xyz=0.0163 -0.007 -0.006 rpy=0 0 -0.55
- joint wheel_back_left_joint: axis 0 0 -1 -> 0 0 1
- joint wheel_back_right_joint: axis 0 0 -1 -> 0 0 1
- joint wheel_front_left_joint: axis 0 0 -1 -> 0 0 1
- joint wheel_front_right_joint: axis 0 0 -1 -> 0 0 1
